Commit message: Fix description reference package path

File: unitree_go1_description/urdf/depthCamera.xacro (robot description, xacro)
@@ -17,5 +17,5 @@
         <origin xyz="0 0 0" rpy="0 0 0"/>
         <geometry>
-          <mesh filename="package://go1_description/models/meshes/depthCamera.dae" scale="1 1 1"/>
+          <mesh filename="package://unitree_go1_description/meshes/depthCamera.dae" scale="1 1 1"/>
         </geometry>
         <material name="black"/>

File: unitree_go1_description/urdf/leg.xacro (robot description, xacro)
@@ -1,5 +1,5 @@
 <?xml version="1.0"?>
 <robot xmlns:xacro="http://www.ros.org/wiki/xacro">
-  <xacro:include filename="$(find go1_description)/models/urdf/transmission.xacro"/>
+  <xacro:include filename="$(find unitree_go1_description)/urdf/transmission.xacro"/>
   <xacro:macro name="leg" params="name mirror mirror_dae front_hind front_hind_dae *origin">
     <joint name="${name}_hip_joint" type="revolute">
@@ -31,5 +31,5 @@
         </xacro:if>
         <geometry>
-          <mesh filename="package://go1_description/models/meshes/hip.dae" scale="1 1 1"/>
+          <mesh filename="package://unitree_go1_description/meshes/hip.dae" scale="1 1 1"/>
         </geometry>
         <material name="silver"/>
@@ -74,8 +74,8 @@
         <geometry>
           <xacro:if value="${mirror_dae == True}">
-            <mesh filename="package://go1_description/models/meshes/thigh.dae" scale="1 1 1"/>
+            <mesh filename="package://unitree_go1_description/meshes/thigh.dae" scale="1 1 1"/>
           </xacro:if>
           <xacro:if value="${mirror_dae == False}">
-            <mesh filename="package://go1_description/models/meshes/thigh_mirror.dae" scale="1 1 1"/>
+            <mesh filename="package://unitree_go1_description/meshes/thigh_mirror.dae" scale="1 1 1"/>
           </xacro:if>
         </geometry>
@@ -106,5 +106,5 @@
         <origin rpy="0 0 0" xyz="0 0 0"/>
         <geometry>
-          <mesh filename="package://go1_description/models/meshes/calf.dae" scale="1 1 1"/>
+          <mesh filename="package://unitree_go1_description/meshes/calf.dae" scale="1 1 1"/>
         </geometry>
         <material name="silver"/>

File: unitree_go1_description/urdf/ros2_control.xacro (robot description, xacro)
@@ -4,5 +4,5 @@
   <xacro:arg name="use_effort_command_interface" default="false"/>
   <xacro:unless value="$(arg use_real_hardware)">
-    <xacro:arg name="ros2_control_config_file" default="$(find go1_description)/config/ros2_controllers.yaml"/>
+    <xacro:arg name="ros2_control_config_file" default="$(find unitree_go1_description)/config/ros2_controllers.yaml"/>
     <xacro:arg name="joint_state_broadcaster_node_name" default="joint_state_broadcaster"/>
   </xacro:unless>

File: unitree_go1_description/urdf/ultraSound.xacro (robot description, xacro)
@@ -17,5 +17,5 @@
         <origin xyz="0 0 0" rpy="0 0 0"/>
         <geometry>
-          <mesh filename="package://go1_description/models/meshes/ultraSound.dae" scale="1 1 1"/>
+          <mesh filename="package://unitree_go1_description/meshes/ultraSound.dae" scale="1 1 1"/>
         </geometry>
         <material name="black"/>

File: unitree_go1_description/urdf/unitree_go1.urdf.xacro (robot description, xacro)
@@ -7,25 +7,17 @@
   <xacro:arg name="enable_sensors_plugin" default="true"/>
   <xacro:arg name="enable_low_resolution_depth" default="true"/>
-  <xacro:include filename="$(find go1_description)/models/urdf/const.xacro"/>
-  <xacro:include filename="$(find go1_description)/models/urdf/materials.xacro"/>
+  <xacro:include filename="$(find unitree_go1_description)/urdf/const.xacro"/>
+  <xacro:include filename="$(find unitree_go1_description)/urdf/materials.xacro"/>
   <xacro:if value="$(arg use_gazebo)">
-    <xacro:include filename="$(find go1_description)/models/urdf/gazebo.xacro"/>
+    <xacro:include filename="$(find unitree_go1_description)/urdf/gazebo.xacro"/>
   </xacro:if>
-  <xacro:include filename="$(find go1_description)/models/urdf/leg.xacro"/>
-  <xacro:include filename="$(find go1_description)/models/urdf/depthCamera.xacro"/>
-  <xacro:include filename="$(find go1_description)/models/urdf/ultraSound.xacro"/>
-  <xacro:include filename="$(find go1_description)/models/urdf/ros2_control.xacro"/>
+  <xacro:include filename="$(find unitree_go1_description)/urdf/leg.xacro"/>
+  <xacro:include filename="$(find unitree_go1_description)/urdf/depthCamera.xacro"/>
+  <xacro:include filename="$(find unitree_go1_description)/urdf/ultraSound.xacro"/>
+  <xacro:include filename="$(find unitree_go1_description)/urdf/ros2_control.xacro"/>
   <!-- Rollover Protection mode will add an additional stick on the top, use "true" or "false" to switch it. -->
   <xacro:property name="rolloverProtection" value="false"/>
   <!-- Debug mode will hung up the robot, use "true" or "false" to switch it. -->
   <xacro:arg name="DEBUG" default="false"/>
-  <xacro:if value="$(arg DEBUG)">
-    <link name="world"/>
-    <joint name="base_static_joint" type="fixed">
-      <origin rpy="0 0 0" xyz="0 0 0"/>
-      <parent link="world"/>
-      <child link="base_link"/>
-    </joint>
-  </xacro:if>
   <link name="base_link">
     <visual>
@@ -45,5 +37,5 @@
       <origin rpy="0 0 0" xyz="0 0 0"/>
       <geometry>
-        <mesh filename="package://go1_description/models/meshes/trunk.dae" scale="1 1 1"/>
+        <mesh filename="package://unitree_go1_description/meshes/trunk.dae" scale="1 1 1"/>
       </geometry>
       <material name="silver"/>

Commit message: Change robot model mesh file path

File: unitree_go1_description/urdf/depthCamera.xacro (robot description, xacro)
@@ -20,5 +20,5 @@
         <origin xyz="0 0 0" rpy="0 0 0"/>
         <geometry>
-          <mesh filename="package://unitree_go1_description/meshes/depthCamera.dae" scale="1 1 1"/>
+          <mesh filename="package://unitree_go1_description/meshes/visual/depthCamera.dae" scale="1 1 1"/>
         </geometry>
         <material name="black"/>

File: unitree_go1_description/urdf/leg.xacro (robot description, xacro)
@@ -34,5 +34,5 @@
         </xacro:if>
         <geometry>
-          <mesh filename="package://unitree_go1_description/meshes/hip.dae" scale="1 1 1"/>
+          <mesh filename="package://unitree_go1_description/meshes/visual/hip.dae" scale="1 1 1"/>
         </geometry>
         <material name="silver"/>
@@ -77,8 +77,8 @@
         <geometry>
           <xacro:if value="${mirror_dae == True}">
-            <mesh filename="package://unitree_go1_description/meshes/thigh.dae" scale="1 1 1"/>
+            <mesh filename="package://unitree_go1_description/meshes/visual/thigh.dae" scale="1 1 1"/>
           </xacro:if>
           <xacro:if value="${mirror_dae == False}">
-            <mesh filename="package://unitree_go1_description/meshes/thigh_mirror.dae" scale="1 1 1"/>
+            <mesh filename="package://unitree_go1_description/meshes/visual/thigh_mirror.dae" scale="1 1 1"/>
           </xacro:if>
         </geometry>
@@ -109,5 +109,5 @@
         <origin rpy="0 0 0" xyz="0 0 0"/>
         <geometry>
-          <mesh filename="package://unitree_go1_description/meshes/calf.dae" scale="1 1 1"/>
+          <mesh filename="package://unitree_go1_description/meshes/visual/calf.dae" scale="1 1 1"/>
         </geometry>
         <material name="silver"/>

File: unitree_go1_description/urdf/ros2_control.xacro (robot description, xacro)
@@ -35,4 +35,5 @@
       </command_interface>
       <command_interface name="velocity">
+        <param name="initial_value">0.0</param>
         <param name="min">${-hip_velocity_max}</param>
         <param name="max">${hip_velocity_max}</param>
@@ -45,5 +46,7 @@
       </xacro:if>
       <state_interface name="position"/>
-      <state_interface name="velocity"/>
+      <state_interface name="velocity">
+        <param name="initial_value">0.0</param>
+      </state_interface>
       <state_interface name="effort"/>
     </joint>
@@ -54,4 +57,5 @@
       </command_interface>
       <command_interface name="velocity">
+        <param name="initial_value">0.0</param>
         <param name="min">${-thigh_velocity_max}</param>
         <param name="max">${thigh_velocity_max}</param>
@@ -64,5 +68,7 @@
       </xacro:if>
       <state_interface name="position"/>
-      <state_interface name="velocity"/>
+      <state_interface name="velocity">
+        <param name="initial_value">0.0</param>
+      </state_interface>
       <state_interface name="effort"/>
     </joint>
@@ -73,4 +79,5 @@
       </command_interface>
       <command_interface name="velocity">
+        <param name="initial_value">0.0</param>
         <param name="min">${-calf_velocity_max}</param>
         <param name="max">${calf_velocity_max}</param>
@@ -83,5 +90,7 @@
       </xacro:if>
       <state_interface name="position"/>
-      <state_interface name="velocity"/>
+      <state_interface name="velocity">
+        <param name="initial_value">0.0</param>
+      </state_interface>
       <state_interface name="effort"/>
     </joint>
@@ -92,4 +101,5 @@
       </command_interface>
       <command_interface name="velocity">
+        <param name="initial_value">0.0</param>
         <param name="min">${-hip_velocity_max}</param>
         <param name="max">${hip_velocity_max}</param>
@@ -102,5 +112,7 @@
       </xacro:if>
       <state_interface name="position"/>
-      <state_interface name="velocity"/>
+      <state_interface name="velocity">
+        <param name="initial_value">0.0</param>
+      </state_interface>
       <state_interface name="effort"/>
     </joint>
@@ -111,4 +123,5 @@
       </command_interface>
       <command_interface name="velocity">
+        <param name="initial_value">0.0</param>
         <param name="min">${-thigh_velocity_max}</param>
         <param name="max">${thigh_velocity_max}</param>
@@ -121,5 +134,7 @@
       </xacro:if>
       <state_interface name="position"/>
-      <state_interface name="velocity"/>
+      <state_interface name="velocity">
+        <param name="initial_value">0.0</param>
+      </state_interface>
       <state_interface name="effort"/>
     </joint>
@@ -130,4 +145,5 @@
       </command_interface>
       <command_interface name="velocity">
+        <param name="initial_value">0.0</param>
         <param name="min">${-calf_velocity_max}</param>
         <param name="max">${calf_velocity_max}</param>
@@ -140,5 +156,7 @@
       </xacro:if>
       <state_interface name="position"/>
-      <state_interface name="velocity"/>
+      <state_interface name="velocity">
+        <param name="initial_value">0.0</param>
+      </state_interface>
       <state_interface name="effort"/>
     </joint>
@@ -149,4 +167,5 @@
       </command_interface>
       <command_interface name="velocity">
+        <param name="initial_value">0.0</param>
         <param name="min">${-hip_velocity_max}</param>
         <param name="max">${hip_velocity_max}</param>
@@ -159,5 +178,7 @@
       </xacro:if>
       <state_interface name="position"/>
-      <state_interface name="velocity"/>
+      <state_interface name="velocity">
+        <param name="initial_value">0.0</param>
+      </state_interface>
       <state_interface name="effort"/>
     </joint>
@@ -168,4 +189,5 @@
       </command_interface>
       <command_interface name="velocity">
+        <param name="initial_value">0.0</param>
         <param name="min">${-thigh_velocity_max}</param>
         <param name="max">${thigh_velocity_max}</param>
@@ -178,5 +200,7 @@
       </xacro:if>
       <state_interface name="position"/>
-      <state_interface name="velocity"/>
+      <state_interface name="velocity">
+        <param name="initial_value">0.0</param>
+      </state_interface>
       <state_interface name="effort"/>
     </joint>
@@ -187,4 +211,5 @@
       </command_interface>
       <command_interface name="velocity">
+        <param name="initial_value">0.0</param>
         <param name="min">${-calf_velocity_max}</param>
         <param name="max">${calf_velocity_max}</param>
@@ -197,5 +222,7 @@
       </xacro:if>
       <state_interface name="position"/>
-      <state_interface name="velocity"/>
+      <state_interface name="velocity">
+        <param name="initial_value">0.0</param>
+      </state_interface>
       <state_interface name="effort"/>
     </joint>
@@ -206,4 +233,5 @@
       </command_interface>
       <command_interface name="velocity">
+        <param name="initial_value">0.0</param>
         <param name="min">${-hip_velocity_max}</param>
         <param name="max">${hip_velocity_max}</param>
@@ -216,5 +244,7 @@
       </xacro:if>
       <state_interface name="position"/>
-      <state_interface name="velocity"/>
+      <state_interface name="velocity">
+        <param name="initial_value">0.0</param>
+      </state_interface>
       <state_interface name="effort"/>
     </joint>
@@ -225,4 +255,5 @@
       </command_interface>
       <command_interface name="velocity">
+        <param name="initial_value">0.0</param>
         <param name="min">${-thigh_velocity_max}</param>
         <param name="max">${thigh_velocity_max}</param>
@@ -235,5 +266,7 @@
       </xacro:if>
       <state_interface name="position"/>
-      <state_interface name="velocity"/>
+      <state_interface name="velocity">
+        <param name="initial_value">0.0</param>
+      </state_interface>
       <state_interface name="effort"/>
     </joint>
@@ -244,4 +277,5 @@
       </command_interface>
       <command_interface name="velocity">
+        <param name="initial_value">0.0</param>
         <param name="min">${-calf_velocity_max}</param>
         <param name="max">${calf_velocity_max}</param>
@@ -254,5 +288,7 @@
       </xacro:if>
       <state_interface name="position"/>
-      <state_interface name="velocity"/>
+      <state_interface name="velocity">
+        <param name="initial_value">0.0</param>
+      </state_interface>
       <state_interface name="effort"/>
     </joint>

File: unitree_go1_description/urdf/ultraSound.xacro (robot description, xacro)
@@ -20,5 +20,5 @@
         <origin xyz="0 0 0" rpy="0 0 0"/>
         <geometry>
-          <mesh filename="package://unitree_go1_description/meshes/ultraSound.dae" scale="1 1 1"/>
+          <mesh filename="package://unitree_go1_description/meshes/visual/ultraSound.dae" scale="1 1 1"/>
         </geometry>
         <material name="black"/>

File: unitree_go1_description/urdf/unitree_go1.urdf.xacro (robot description, xacro)
@@ -41,5 +41,5 @@
       <origin rpy="0 0 0" xyz="0 0 0"/>
       <geometry>
-        <mesh filename="package://unitree_go1_description/meshes/trunk.dae" scale="1 1 1"/>
+        <mesh filename="package://unitree_go1_description/meshes/visual/trunk.dae" scale="1 1 1"/>
       </geometry>
       <material name="silver"/>
