Commit message: reflect the pointed out issues

File: unitree_go1_description/urdf/go1_livox_mount.xacro (robot description, xacro)
@@ -1,31 +1,4 @@
 <?xml version="1.0" ?>
 <robot name="go1_livox_mount" xmlns:xacro="http://www.ros.org/wiki/xacro">
-<!--
-<xacro:include filename="$(find unitree_go1_description_description)/urdf/materials.xacro" />
-<xacro:include filename="$(find unitree_go1_description_description)/urdf/Go1_livox_mouont.trans" />
-<xacro:include filename="$(find unitree_go1_description_description)/urdf/Go1_livox_mouont.gazebo" />
--->
-<!--
-<link name="base_link">
-  <inertial>
-    <origin xyz="-0.000795843710238667 -0.0017600633360694503 0.026855412423998835" rpy="0 0 0"/>
-    <mass value="19.412938243918365"/>
-    <inertia ixx="0.055081" iyy="0.111616" izz="0.157" ixy="0.001148" iyz="-0.000287" ixz="0.000258"/>
-  </inertial>
-  <visual>
-    <origin xyz="0 0 0" rpy="0 0 0"/>
-    <geometry>
-      <mesh filename="file://$(find unitree_go1_description_description)/meshes/base_link.stl" scale="0.001 0.001 0.001"/>
-    </geometry>
-    <material name="silver"/>
-  </visual>
-  <collision>
-    <origin xyz="0 0 0" rpy="0 0 0"/>
-    <geometry>
-      <mesh filename="file://$(find unitree_go1_description_description)/meshes/base_link.stl" scale="0.001 0.001 0.001"/>
-    </geometry>
-  </collision>
-</link>
--->
 <link name="sensor_mount_link">
   <inertial>
@@ -37,5 +10,5 @@
     <origin xyz="-0.044 0 -0.057" rpy="0 0 0"/>
     <geometry>
-      <mesh filename="file://$(find unitree_go1_description_description)/meshes/visual/units/sensor_mount.stl" scale="0.001 0.001 0.001"/>
+      <mesh filename="file://$(find unitree_go1_description)/meshes/visual/units/sensor_mount.stl" scale="0.001 0.001 0.001"/>
     </geometry>
     <material name="silver"/>
@@ -44,5 +17,5 @@
     <origin xyz="-0.044 0 -0.057" rpy="0 0 0"/>
     <geometry>
-      <mesh filename="file://$(find unitree_go1_description_description)/meshes/visual/units/sensor_mount.stl" scale="0.001 0.001 0.001"/>
+      <mesh filename="file://$(find unitree_go1_description)/meshes/visual/units/sensor_mount.stl" scale="0.001 0.001 0.001"/>
     </geometry>
   </collision>
@@ -62,6 +35,6 @@
   <origin xyz="0 0 0.170" rpy="3.1415926 0 0"/>
   <parent link="sensor_mount_link"/>
-  <child link="mid360_link"/>
+  <child link="livox_frame"/>
 </joint>
-<link name="mid360_link"/>
+<link name="livox_frame"/>
 </robot>

File: unitree_go1_description/urdf/tc24_unitree_go1.urdf.xacro (robot description, xacro)
@@ -162,6 +162,3 @@
     <origin rpy="0 0 0" xyz="0.2747 0.0 -0.0088"/>
   </xacro:ultraSound>
-  <xacro:backpack_sensor_unit name="tc23" parent="base_link">
-    <origin rpy="0 0 0" xyz="0 0 0"/>
-  </xacro:backpack_sensor_unit>
 </robot>

Commit message: rename link imu_link --> witmotion_imu_link

File: unitree_go1_description/urdf/go1_livox_mount.xacro (robot description, xacro)
@@ -26,10 +26,10 @@
   <child link="sensor_mount_link"/>
 </joint>
-<joint name="mount_to_imu_joint" type="fixed">
+<joint name="mount_to_witmotion_joint" type="fixed">
   <origin xyz="0 0 0.105" rpy="0 0 0"/>
   <parent link="sensor_mount_link"/>
-  <child link="imu_link"/>
+  <child link="witmotion_imu_link"/>
 </joint>
-<link name="imu_link"/>
+<link name="witmotion_imu_link"/>
 <joint name="mount_to_mid360_joint" type="fixed">
   <origin xyz="0 0 0.170" rpy="3.1415926 0 0"/>

Commit message: add stl model for collision

File: unitree_go1_description/urdf/go1_livox_mount.xacro (robot description, xacro)
@@ -17,5 +17,5 @@
     <origin xyz="-0.044 0 -0.057" rpy="0 0 0"/>
     <geometry>
-      <mesh filename="file://$(find unitree_go1_description)/meshes/visual/units/sensor_mount.stl" scale="0.001 0.001 0.001"/>
+      <mesh filename="file://$(find unitree_go1_description)/meshes/visual/units/sensor_mount_for_collision.stl" scale="0.001 0.001 0.001"/>
     </geometry>
   </collision>

Commit message: change the model foile to more lighter

File: unitree_go1_description/urdf/go1_livox_mount.xacro (robot description, xacro)
@@ -8,14 +8,14 @@
   </inertial>
   <visual>
-    <origin xyz="-0.044 0 -0.057" rpy="0 0 0"/>
+    <origin xyz="0 0 0" rpy="0 0 0"/>
     <geometry>
-      <mesh filename="file://$(find unitree_go1_description)/meshes/visual/units/sensor_mount.stl" scale="0.001 0.001 0.001"/>
+      <mesh filename="file://$(find unitree_go1_description)/meshes/visual/units/sensor_mount.dae" scale="1 1 1"/>
     </geometry>
     <material name="silver"/>
   </visual>
   <collision>
-    <origin xyz="-0.044 0 -0.057" rpy="0 0 0"/>
+    <origin xyz="0 0 0" rpy="0 0 0"/>
     <geometry>
-      <mesh filename="file://$(find unitree_go1_description)/meshes/visual/units/sensor_mount_for_collision.stl" scale="0.001 0.001 0.001"/>
+      <mesh filename="file://$(find unitree_go1_description)/meshes/visual/units/sensor_mount_for_collision.stl" scale="1 1 1"/>
     </geometry>
   </collision>
